Commit message: fix
Signed-off-by: Amadeusz Szymko <amadeusz.szymko@put.poznan.pl>

File: abb_irb_120_resource/urdf/irb_120_macro.xacro (robot description, xacro)
@@ -30,5 +30,5 @@
     <xacro:property name="l7_dl" value="-400" />
     <xacro:property name="l7_ul" value="400" />
-    <xacro:property name="e_trans" value="0.0 0.0 0.012" />
+    <xacro:property name="e_trans" value="0.0 0.0 0.028" />
     <xacro:property name="e_rot" value="0.0 0.0 0.0" />
     <xacro:property name="e_dl" value="" />

Commit message: feat: demo settings
Signed-off-by: Amadeusz Szymko <amadeusz.szymko@put.poznan.pl>

File: abb_irb_120_resource/urdf/irb_120_macro.xacro (robot description, xacro)
@@ -30,5 +30,5 @@
     <xacro:property name="l7_dl" value="-400" />
     <xacro:property name="l7_ul" value="400" />
-    <xacro:property name="e_trans" value="0.0 0.0 0.028" />
+    <xacro:property name="e_trans" value="0.0 0.0 0.2" />
     <xacro:property name="e_rot" value="0.0 0.0 0.0" />
     <xacro:property name="e_dl" value="" />
